Commit message: all the 2 cameras, lidar, and 5 sensors location have been move their rightful location

File: src/oil_palm_harvester_description/urdf/oil_palm_harvester_estimated.urdf (robot description, URDF)
Before this commit: robot oil_palm_harvester_estimated, 29 links, 28 joints
Links:
- added link front_depth_camera_link, mass 0.3500; collision box size=0.12 0.05 0.05; visual mesh filename=package://oil_palm_harvester_description/meshes/visual/dept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 scale=1 1 1
- added link front_depth_camera_optical_frame
- added link front_sensor_mount_link, mass 1.0; collision box size=0.30 0.30 0.16; visual box size=0.30 0.30 0.16
- link cutting_arm_base_link: geometry collision box size=0.35 0.34 0.34; visual mesh filename=package://oil_palm_harvester_description/meshes/visual/cutt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 scale=0.5 1 1
- link cutting_arm_extension_link: geometry collision box size=0.475 0.2 0.2; visual mesh filename=package://oil_palm_harvester_description/meshes/visual/cutt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 scale=0.5 1 1
- link cutting_tool_link: geometry collision box size=0.225 0.22 0.18; visual mesh filename=package://oil_palm_harvester_description/meshes/visual/cutt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 scale=0.5 1 1
Joints:
- added joint front_depth_camera_joint: type fixed, parent front_sensor_mount_link, child front_depth_camera_link, origin xyz=0.04 -0.09 0.13 rpy=0 0 0
- added joint front_depth_camera_optical_joint: type fixed, parent front_depth_camera_link, child front_depth_camera_optical_frame, origin xyz=0 0 0 rpy=-1.5707963267948966 0 -1.5707963267948966
- added joint front_sensor_mount_joint: type fixed, parent platform_mount_link, child front_sensor_mount_link, origin xyz=0.45 0 0.32 rpy=0 0 0
- joint center_range_sensor_joint: origin xyz=0.43 0 0.1 rpy=0 0 0 -> xyz=0.18 0 0.115 rpy=0 0 0; parent c_channel_platform_link -> front_sensor_mount_link
- joint cutting_arm_extension_joint: limit lower=0.0 upper=0.75 effort=2200 velocity=0.2 -> lower=0.0 upper=0.375 effort=2200 velocity=0.2; origin xyz=0.62 0 0 rpy=0 0 0 -> xyz=0.31 0 0 rpy=0 0 0
- joint cutting_tool_fixed_joint: origin xyz=0.92 0 0 rpy=0 0 0 -> xyz=0.46 0 0 rpy=0 0 0
- joint left_side_range_sensor_joint: origin xyz=0.05 0.95 0.1 rpy=0 0 -1.5707963267948966 -> xyz=0.95 0.95 0.1 rpy=0 0 -1.5707963267948966
- joint platform_depth_camera_joint: origin xyz=-0.42 0 0.72 rpy=0 -0.12 0 -> xyz=0.125 0 0.12 rpy=0 0.22 0.13; parent c_channel_platform_link -> cutting_arm_base_link
- joint right_side_range_sensor_joint: origin xyz=0.05 -0.95 0.1 rpy=0 0 1.5707963267948966 -> xyz=0.95 -0.95 0.1 rpy=0 0 1.5707963267948966
- joint vehicle_lidar_joint: origin xyz=-1.3 0 2.72 rpy=0 0 0 -> xyz=0.125 0 0.41 rpy=0 0 0; parent base_link -> cutting_arm_base_link

File: src/oil_palm_harvester_description/urdf/oil_palm_harvester_kinematic.urdf (robot description, URDF)
Before this commit: robot oil_palm_harvester_estimated, 29 links, 28 joints
Links:
- added link front_depth_camera_link, mass 0.3500; collision box size=0.12 0.05 0.05; visual mesh filename=package://oil_palm_harvester_description/meshes/visual/dept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 scale=1 1 1
- added link front_depth_camera_optical_frame
- added link front_sensor_mount_link, mass 1.0; collision box size=0.30 0.30 0.16; visual box size=0.30 0.30 0.16
- link cutting_arm_base_link: geometry collision box size=0.35 0.34 0.34; visual mesh filename=package://oil_palm_harvester_description/meshes/visual/cutt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 scale=0.5 1 1
- link cutting_arm_extension_link: geometry collision box size=0.475 0.2 0.2; visual mesh filename=package://oil_palm_harvester_description/meshes/visual/cutt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 scale=0.5 1 1
- link cutting_tool_link: geometry collision box size=0.225 0.22 0.18; visual mesh filename=package://oil_palm_harvester_description/meshes/visual/cutt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 scale=0.5 1 1
Joints:
- added joint front_depth_camera_joint: type fixed, parent front_sensor_mount_link, child front_depth_camera_link, origin xyz=0.2 0.0 0.00 rpy=0 0 0
- added joint front_depth_camera_optical_joint: type fixed, parent front_depth_camera_link, child front_depth_camera_optical_frame, origin xyz=0 0 0 rpy=-1.5707963267948966 0 -1.5707963267948966
- added joint front_sensor_mount_joint: type fixed, parent platform_mount_link, child front_sensor_mount_link, origin xyz=0.55 0 0.2 rpy=0 0 0
- joint center_range_sensor_joint: origin xyz=0.43 0 0.1 rpy=0 0 0 -> xyz=0.0 0 0.115 rpy=0 0 0; parent c_channel_platform_link -> front_sensor_mount_link
- joint cutting_arm_extension_joint: limit lower=0.0 upper=0.75 effort=2200 velocity=0.2 -> lower=0.0 upper=0.375 effort=2200 velocity=0.2; origin xyz=0.62 0 0 rpy=0 0 0 -> xyz=0.31 0 0 rpy=0 0 0
- joint cutting_tool_fixed_joint: origin xyz=0.92 0 0 rpy=0 0 0 -> xyz=0.46 0 0 rpy=0 0 0
- joint left_side_range_sensor_joint: origin xyz=0.05 0.95 0.1 rpy=0 0 -1.5707963267948966 -> xyz=0.95 0.95 0.1 rpy=0 0 -1.5707963267948966
- joint platform_depth_camera_joint: origin xyz=-0.42 0 0.72 rpy=0 -0.12 0 -> xyz=0.125 0 0.25 rpy=0 0.0 0.0; parent c_channel_platform_link -> cutting_arm_base_link
- joint right_side_range_sensor_joint: origin xyz=0.05 -0.95 0.1 rpy=0 0 1.5707963267948966 -> xyz=0.95 -0.95 0.1 rpy=0 0 1.5707963267948966
- joint vehicle_lidar_joint: origin xyz=-1.3 0 2.72 rpy=0 0 0 -> xyz=0 0 0.3 rpy=0 0 0; parent base_link -> cutting_arm_base_link
