Commit message: All 10 movable joints use rate-limited kinematic control at 20 Hz. Updated the project documentation to the current working state

File: src/oil_palm_harvester_description/urdf/oil_palm_harvester_kinematic.urdf (robot description, URDF)
Before this commit: robot oil_palm_harvester_estimated, 32 links, 31 joints
Links:
- added link cutting_tool_left_range_sensor_link, mass 0.0100; visual mesh filename=package://oil_palm_harvester_description/meshes/visual/rang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 scale=1 1 1
Joints:
- added joint cutting_tool_left_range_sensor_joint: type fixed, parent cutting_tool_link, child cutting_tool_left_range_sensor_link, origin xyz=0.10 0.12 0.00 rpy=0 0 0
